File: Projeto Base/Projeto-Natal-2023-Base/Projeto-Natal-2023-Base.kicad_pcb (KiCad board)
At the start: 2 copper layers, 40 parts, among them U1 STM8S003F3P

Commit message: trocando mcu para ch32v003f4p6
Parts:
- removed C4: 10uF, Capacitor_SMD:C_0805_2012Metric_Pad1.18x1.45mm_HandSolder
- removed C5: 100nF, Capacitor_SMD:C_0603_1608Metric_Pad1.08x0.95mm_HandSolder
- U1: value STM8S003F3P -> CH32V003F4P6
- moved C3 21.9 mm to (168.3, 119.2)
- moved R10 20.1 mm to (168.3, 121.7)
- moved R11 20.1 mm to (168.3, 124.2)
- moved C2 17.6 mm to (168.5, 127.0)
- moved U1 11.7 mm to (161.8, 123.7)
Connections:
- C2 pad 1: Net-(U1-VCAP) -> +3V3
- C3 pad 2: Net-(U1-VCAP) -> +3V3
- R10 pad 1: LED9 -> Net-(U1-PC0)
- R10 pad 2: Net-(U1-PC6) -> LED11
- R11 pad 1: LED10 -> Net-(U1-PC1)
- R11 pad 2: Net-(U1-PC7) -> LED11
- R12 pad 1: Net-(U1-PD1) -> Net-(U1-PC2)
- R13 pad 1: Net-(U1-PD2) -> Net-(U1-PC3)
- R14 pad 1: Net-(U1-PD3) -> Net-(U1-PC4)
- R15 pad 1: Net-(U1-PD4) -> Net-(U1-PC5)
- R16 pad 1: Net-(U1-PD5) -> Net-(U1-PC6)
- R17 pad 1: Net-(U1-PD6) -> Net-(U1-PC7)
- R2 pad 2: Net-(U1-PA1) -> Net-(U1-OSC_OUT/PA2)
- R3 pad 2: Net-(U1-PA2) -> Net-(U1-PD0)
- R4 pad 2: Net-(U1-PA3) -> Net-(U1-PD1)
- R5 pad 2: Net-(U1-PB4) -> Net-(U1-PD2)
- R6 pad 2: Net-(U1-PB5) -> Net-(U1-PD3)
- R7 pad 2: Net-(U1-PC3) -> Net-(U1-PD4)
- R8 pad 2: Net-(U1-PC4) -> Net-(U1-PD5)
- R9 pad 2: Net-(U1-PC5) -> Net-(U1-PD6)
- U1 pad 10: Net-(U1-PA3) -> Net-(U1-PC0)
- U1 pad 11: Net-(U1-PB5) -> Net-(U1-PC1)
- U1 pad 12: Net-(U1-PB4) -> Net-(U1-PC2)
- U1 pad 5: Net-(U1-PA1) -> unconnected-(U1-OSC_IN/PA1-Pad5)
- U1 pad 6: Net-(U1-PA2) -> Net-(U1-OSC_OUT/PA2)
- U1 pad 8: Net-(U1-VCAP) -> Net-(U1-PD0)

Commit message: Adicionando conector de SWIO
Parts:
- added J1: Conn_01x03_Pin, Connector_PinHeader_2.54mm:PinHeader_1x03_P2.54mm_Vertical, F.Cu at (181.0, 120.7)
- moved BT1 5.67 mm to (149.2, 84.5)
Connections:
- R2 pad 2: Net-(U1-OSC_OUT/PA2) -> Net-(U1-OSC_IN/PA1)
- R3 pad 2: Net-(U1-PD0) -> Net-(U1-OSC_OUT/PA2)
- R4 pad 2: Net-(U1-PD1) -> Net-(U1-PD0)
- U1 pad 18: Net-(U1-PD1) -> SWIO
- U1 pad 5: unconnected-(U1-OSC_IN/PA1-Pad5) -> Net-(U1-OSC_IN/PA1)
Changed lines of the file:
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@@
   (net 22 "Net-(U1-PC6)")
   (net 23 "Net-(U1-PC7)")
-  (net 24 "Net-(U1-PD1)")
+  (net 24 "Net-(U1-OSC_IN{slash}PA1)")
   (net 25 "Net-(U1-PD2)")
   (net 26 "Net-(U1-PD3)")
@@
   (net 34 "Net-(U1-PC1)")
   (net 35 "Net-(U1-PC2)")
-  (net 36 "unconnected-(U1-OSC_IN{slash}PA1-Pad5)")
+  (net 36 "SWIO")
   (footprint "LED_THT:LED_D5.0mm" (layer "F.Cu")
     (at 152.1925 114.26)
@@
       (net 3 "LED1") (pintype "passive"))
     (pad "2" smd roundrect (at 0.9125 0) (size 0.975 0.95) (layers "F.Cu" "F.Paste" "F.Mask") (roundrect_rratio 0.25)
-      (net 31 "Net-(U1-OSC_OUT{slash}PA2)") (pintype "passive"))
+      (net 24 "Net-(U1-OSC_IN{slash}PA1)") (pintype "passive"))
     (model "${KICAD6_3DMODEL_DIR}/Resistor_SMD.3dshapes/R_0603_1608Metric.wrl"
       (offset (xyz 0 0 0))
@@
     )
   )
+  (footprint "Connector_PinHeader_2.54mm:PinHeader_1x03_P2.54mm_Vertical" (layer "F.Cu")
+    (at 180.975 120.65)
+    (descr "Through hole straight pin header, 1x03, 2.54mm pitch, single row")
+    (tags "Through hole pin header THT 1x03 2.54mm single row")
+    (property "Sheetfile" "Projeto-Natal-2023-Base.kicad_sch")
+    (property "Sheetname" "")
+    (property "ki_description" "Generic connector, single row, 01x03, script generated")
+    (property "ki_keywords" "connector")
+    (attr through_hole)
+    (fp_text reference "J1" (at 0 -2.33) (layer "F.SilkS")
+        (effects (font (size 1 1) (thickness 0.15)))
+    )
+    (fp_text value "Conn_01x03_Pin" (at 0 7.41) (layer "F.Fab")
+        (effects (font (size 1 1) (thickness 0.15)))
+    )
+    (fp_text user "${REFERENCE}" (at 0 2.54 90) (layer "F.Fab")
+        (effects (font (size 1 1) (thickness 0.15)))
+    )
+    (fp_line (start -1.33 -1.33) (end 0 -1.33)
+      (stroke (width 0.12) (type solid)) (layer "F.SilkS"))
+    (fp_line (start -1.33 0) (end -1.33 -1.33)
+      (stroke (width 0.12) (type solid)) (layer "F.SilkS"))
+    (fp_line (start -1.33 1.27) (end -1.33 6.41)
+      (stroke (width 0.12) (type solid)) (layer "F.SilkS"))
+    (fp_line (start -1.33 1.27) (end 1.33 1.27)
+      (stroke (width 0.12) (type solid)) (layer "F.SilkS"))
+    (fp_line (start -1.33 6.41) (end 1.33 6.41)
+      (stroke (width 0.12) (type solid)) (layer "F.SilkS"))
+    (fp_line (start 1.33 1.27) (end 1.33 6.41)
+      (stroke (width 0.12) (type solid)) (layer "F.SilkS"))
+    (fp_line (start -1.8 -1.8) (end -1.8 6.85)
+      (stroke (width 0.05) (type solid)) (layer "F.CrtYd"))
+    (fp_line (start -1.8 6.85) (end 1.8 6.85)
+      (stroke (width 0.05) (type solid)) (layer "F.CrtYd"))
+    (fp_line (start 1.8 -1.8) (end -1.8 -1.8)
+      (stroke (width 0.05) (type solid)) (layer "F.CrtYd"))
+    (fp_line (start 1.8 6.85) (end 1.8 -1.8)
+      (stroke (width 0.05) (type solid)) (layer "F.CrtYd"))
+    (fp_line (start -1.27 -0.635) (end -0.635 -1.27)
+      (stroke (width 0.1) (type solid)) (layer "F.Fab"))
+    (fp_line (start -1.27 6.35) (end -1.27 -0.635)
+      (stroke (width 0.1) (type solid)) (layer "F.Fab"))
+    (fp_line (start -0.635 -1.27) (end 1.27 -1.27)
+      (stroke (width 0.1) (type solid)) (layer "F.Fab"))
+    (fp_line (start 1.27 -1.27) (end 1.27 6.35)
+      (stroke (width 0.1) (type solid)) (layer "F.Fab"))
+    (fp_line (start 1.27 6.35) (end -1.27 6.35)
+      (stroke (width 0.1) (type solid)) (layer "F.Fab"))
+    (pad "1" thru_hole rect (at 0 0) (size 1.7 1.7) (drill 1) (layers "*.Cu" "*.Mask")
+      (net 1 "+3V3") (pinfunction "Pin_1") (pintype "passive"))
+    (pad "2" thru_hole oval (at 0 2.54) (size 1.7 1.7) (drill 1) (layers "*.Cu" "*.Mask")
+      (net 2 "GND") (pinfunction "Pin_2") (pintype "passive"))
+    (pad "3" thru_hole oval (at 0 5.08) (size 1.7 1.7) (drill 1) (layers "*.Cu" "*.Mask")
+      (net 36 "SWIO") (pinfunction "Pin_3") (pintype "passive"))
+    (model "${KICAD6_3DMODEL_DIR}/Connector_PinHeader_2.54mm.3dshapes/PinHeader_1x03_P2.54mm_Vertical.wrl"
+      (offset (xyz 0 0 0))
+      (scale (xyz 1 1 1))
+      (rotate (xyz 0 0 0))
+    )
+  )
   (footprint "LED_THT:LED_D5.0mm" (layer "F.Cu")
     (at 144.6925 114.26)
@@
   )
   (footprint "Battery:BatteryHolder_Keystone_3002_1x2032" (layer "F.Cu")
-    (at 143.5925 83.767512)
+    (at 149.225 84.455)
     (descr "https://www.tme.eu/it/Document/a823211ec201a9e209042d155fe22d2b/KEYS2996.pdf")
     (tags "BR2016 CR2016 DL2016 BR2020 CL2020 BR2025 CR2025 DL2025 DR2032 CR2032 DL2032")
@@
       (net 30 "Net-(U1-NRST{slash}PD7)") (pinfunction "NRST/PD7") (pintype "input"))
     (pad "5" smd roundrect (at -2.8625 -0.325) (size 1.475 0.4) (layers "F.Cu" "F.Paste" "F.Mask") (roundrect_rratio 0.25)
-      (net 36 "unconnected-(U1-OSC_IN{slash}PA1-Pad5)") (pinfunction "OSC_IN/PA1") (pintype "input"))
+      (net 24 "Net-(U1-OSC_IN{slash}PA1)") (pinfunction "OSC_IN/PA1") (pintype "input"))
     (pad "6" smd roundrect (at -2.8625 0.325) (size 1.475 0.4) (layers "F.Cu" "F.Paste" "F.Mask") (roundrect_rratio 0.25)
       (net 31 "Net-(U1-OSC_OUT{slash}PA2)") (pinfunction "OSC_OUT/PA2") (pintype "input"))
@@
       (net 23 "Net-(U1-PC7)") (pinfunction "PC7") (pintype "bidirectional"))
     (pad "18" smd roundrect (at 2.8625 -1.625) (size 1.475 0.4) (layers "F.Cu" "F.Paste" "F.Mask") (roundrect_rratio 0.25)
-      (net 24 "Net-(U1-PD1)") (pinfunction "PD1") (pintype "bidirectional"))
+      (net 36 "SWIO") (pinfunction "PD1") (pintype "bidirectional"))
     (pad "19" smd roundrect (at 2.8625 -2.275) (size 1.475 0.4) (layers "F.Cu" "F.Paste" "F.Mask") (roundrect_rratio 0.25)
       (net 25 "Net-(U1-PD2)") (pinfunction "PD2") (pintype "bidirectional"))
@@
       (net 7 "LED2") (pintype "passive"))
     (pad "2" smd roundrect (at 0.9125 0) (size 0.975 0.95) (layers "F.Cu" "F.Paste" "F.Mask") (roundrect_rratio 0.25)
-      (net 32 "Net-(U1-PD0)") (pintype "passive"))
+      (net 31 "Net-(U1-OSC_OUT{slash}PA2)") (pintype "passive"))
     (model "${KICAD6_3DMODEL_DIR}/Resistor_SMD.3dshapes/R_0603_1608Metric.wrl"
       (offset (xyz 0 0 0))
@@
       (net 11 "LED3") (pintype "passive"))
     (pad "2" smd roundrect (at 0.9125 0) (size 0.975 0.95) (layers "F.Cu" "F.Paste" "F.Mask") (roundrect_rratio 0.25)
-      (net 24 "Net-(U1-PD1)") (pintype "passive"))
+      (net 32 "Net-(U1-PD0)") (pintype "passive"))
     (model "${KICAD6_3DMODEL_DIR}/Resistor_SMD.3dshapes/R_0603_1608Metric.wrl"
       (offset (xyz 0 0 0))
